Commit message: add point cloud to simulation

File: src/gelsight_simulation_ros/gelsight_description/urdf/gelsight_sensor.xacro (robot description, xacro)
@@ -2,5 +2,140 @@
 <robot xmlns:xacro="http://ros.org/wiki/xacro">
     <xacro:include filename="$(find gelsight_description)/urdf/gs_mini_spectre.xacro"/>
-    <!-- ++++++++++++++++++++++++++++++ Camera simulation +++++++++++++++++++++++++++++++++++-->
+  <xacro:macro name="gelsight_sensor" params="parent">
+    <link name="gs_kinova_holder_link">
+      <visual>
+        <geometry>
+          <mesh filename="package://gelsight_description/meshes/remain/gs_holder.stl" scale="0.001 0.001 0.001"/>
+        </geometry>
+        <material name="">
+          <color rgba="1 1 1 1"/>
+        </material>
+      </visual>
+      <inertial>
+        <mass value="0.1"/>
+        <origin xyz="0 0 0" rpy="0 0 0"/>
+        <inertia ixx="0.001" ixy="0.0" ixz="0.0"
+                 iyy="0.001" iyz="0.0"
+                 izz="0.001"/>
+      </inertial>
+    </link>
+    <link name="gs_base_link">
+      <visual>
+        <geometry>
+          <mesh filename="package://gelsight_description/meshes/remain/gs_base.stl" scale="0.001 0.001 0.001"/>
+        </geometry>
+        <material name="">
+          <color rgba="0.5 0.5 0.5 1"/>
+        </material>
+      </visual>
+      <inertial>
+        <mass value="0.1"/>
+        <origin xyz="0 0 0" rpy="0 0 0"/>
+        <inertia ixx="0.001" ixy="0.0" ixz="0.0"
+                 iyy="0.001" iyz="0.0"
+                 izz="0.001"/>
+      </inertial>
+    </link>
+    <link name="gs_cap_link">
+      <visual>
+        <geometry>
+          <mesh filename="package://gelsight_description/meshes/remain/gs_cap.stl" scale="0.001 0.001 0.001"/>
+        </geometry>
+        <material name="">
+          <color rgba="0 0 0 1"/>
+        </material>
+      </visual>
+      <inertial>
+        <mass value="0.1"/>
+        <origin xyz="0 0 0" rpy="0 0 0"/>
+        <inertia ixx="0.001" ixy="0.0" ixz="0.0"
+                 iyy="0.001" iyz="0.0"
+                 izz="0.001"/>
+      </inertial>
+    </link>
+    <!-- <link name="gs_gel_link">
+      <visual>
+        <geometry>
+          <mesh filename="package://gelsight_description/meshes/remain/gs_gel.stl" scale="0.001 0.001 0.001"/>
+        </geometry>
+        <material name="">
+            <color rgba="0.8 0.8 1.0 0.0"/>
+        </material>
+      </visual>
+      <inertial>
+        <mass value="0.1"/>
+        <origin xyz="0 0 0" rpy="0 0 0"/>
+        <inertia ixx="0.001" ixy="0.0" ixz="0.0"
+                 iyy="0.001" iyz="0.0"
+                 izz="0.001"/>
+      </inertial>
+    </link> -->
+      <link name="gs_gel_link">
+      <inertial>
+        <mass value="0.1"/>
+        <origin xyz="0 0 0" rpy="0 0 0"/>
+        <inertia ixx="0.001" ixy="0.0" ixz="0.0"
+                iyy="0.001" iyz="0.0"
+                izz="0.001"/>
+      </inertial>
+    </link>
+    <!-- <link name="gs_glass_link">
+      <visual>
+        <geometry>
+          <mesh filename="package://gelsight_description/meshes/remain/gs_glass.stl" scale="0.001 0.001 0.001"/>
+        </geometry>
+        <material name="">
+            <color rgba="1.0 1.0 1.0 0.3"/>
+        </material>
+      </visual>
+      <inertial>
+        <mass value="0.1"/>
+        <origin xyz="0 0 0" rpy="0 0 0"/>
+        <inertia ixx="0.001" ixy="0.0" ixz="0.0"
+                 iyy="0.001" iyz="0.0"
+                 izz="0.001"/>
+      </inertial>
+    </link> -->
+    <joint name="gs_holder_joint" type="fixed">
+      <parent link="${parent}"/>
+      <child link="gs_kinova_holder_link"/>
+      <origin xyz="-0.0380 -0.038 0" rpy="0 0 0"/>
+    </joint>
+    <joint name="gs_base_joint" type="fixed">
+      <parent link="${parent}"/>
+      <child link="gs_base_link"/>
+      <origin xyz="-0.014 -0.016 0" rpy="0 0 0"/>
+    </joint>
+    <joint name="gs_cap_joint" type="fixed">
+      <parent link="${parent}"/>
+      <child link="gs_cap_link"/>
+      <origin xyz="-0.0144 -0.016 0" rpy="0 0 0"/>
+    </joint>
+    <joint name="gs_gel_joint" type="fixed">
+      <parent link="${parent}"/>
+      <child link="gs_gel_link"/>
+      <origin xyz="-0.0115 -0.01386 0" rpy="0 0 0"/>
+    </joint>
+      <!-- +++++++++++++++++++++++camera link+++++++++++++++++++++++++++++ -->
+        <link name="gs_camera_link">
+      <visual>
+        <geometry>
+          <mesh filename="package://gelsight_description/meshes/remain/gs_glass.stl" scale="0.000001 0.0000001 0.0000001"/>
+        </geometry>
+      </visual>
+    </link>
+    <joint name="gs_camera_joint" type="fixed">
+      <parent link="gs_gel_link"/>
+      <child link="gs_camera_link"/>
+      <origin xyz="0.012 0.0143 0.035" rpy="0 ${-pi/2} ${pi}"/>
+      <!-- <origin xyz="0.012 0.0143 0.035" rpy="0 0 0"/> -->
+    </joint>
+    <link name="gs_camera_pcloud"/>
+    <joint name="gs_camera_pcloud_joint" type="fixed">
+      <parent link="gs_gel_link"/>
+      <child link="gs_camera_pcloud"/>
+      <origin xyz="0.012 0.0143 0.035" rpy="0 0 ${pi/2}"/>
+    </joint>
+     <!-- ++++++++++++++++++++++++++++++ Camera simulation +++++++++++++++++++++++++++++++++++-->
      <xacro:macro name="gelsight_camera" params="parent">
     <gazebo reference="${parent}">
@@ -12,5 +147,5 @@
         <topic>/depth_camera</topic>
         <camera name="head">
-          <horizontal_fov>1.309</horizontal_fov>
+          <horizontal_fov>0.959931</horizontal_fov>
           <image>
             <width>320</width>
@@ -36,5 +171,5 @@
           <depthImageInfoTopicName>/gelsight/depth/camera_info</depthImageInfoTopicName>
           <pointCloudTopicName>/gelsight/depth/points</pointCloudTopicName>
-          <frameName>${parent}</frameName>
+          <frameName>gs_camera_pcloud</frameName>
           <pointCloudCutoff>0.0</pointCloudCutoff>
           <distortionK1>0</distortionK1>
@@ -52,166 +187,5 @@
     </gazebo>
   </xacro:macro>
-   <!-- <xacro:macro name="gelsight_camera" params="parent">
-  <gazebo reference="${parent}">
-    <sensor type="camera" name="gelsight_rgb_camera">
-      <pose>0 0 0 0 0 0</pose>
-      <always_on>1</always_on>
-      <update_rate>30.0</update_rate>
-      <visualize>1</visualize>
-      <camera name="main_camera">
-     75 degrees of fov
-        <horizontal_fov>1.309</horizontal_fov>
-        <image>
-          <width>320</width>
-          <height>240</height>
-          <format>R8G8B8</format>
-        </image>
-        <clip>
-          <near>0.001</near>
-          <far>0.1</far>
-        </clip>
-      </camera>
-      <plugin name="gelsight_rgb_camera_controller" filename="libgazebo_ros_camera.so">
-        <alwaysOn>true</alwaysOn>
-        <updateRate>30.0</updateRate>
-        <cameraName>gelsight_rgb</cameraName>
-        <imageTopicName>/gelsight/image/image_raw</imageTopicName>
-        <cameraInfoTopicName>/gelsight/camera_info</cameraInfoTopicName>
-        <frameName>${parent}</frameName>
-      </plugin>
-    </sensor>
-  </gazebo>
-</xacro:macro> -->
     <!-- +++++++++++++++++++++++++++++++++++++++++++++++++++++++++++++++++++++++++++++++++++ -->
-  <xacro:macro name="gelsight_sensor" params="parent">
-    <link name="gs_kinova_holder_link">
-      <visual>
-        <geometry>
-          <mesh filename="package://gelsight_description/meshes/remain/gs_holder.stl" scale="0.001 0.001 0.001"/>
-        </geometry>
-        <material name="">
-          <color rgba="1 1 1 1"/>
-        </material>
-      </visual>
-      <inertial>
-        <mass value="0.1"/>
-        <origin xyz="0 0 0" rpy="0 0 0"/>
-        <inertia ixx="0.001" ixy="0.0" ixz="0.0"
-                 iyy="0.001" iyz="0.0"
-                 izz="0.001"/>
-      </inertial>
-    </link>
-    <link name="gs_base_link">
-      <visual>
-        <geometry>
-          <mesh filename="package://gelsight_description/meshes/remain/gs_base.stl" scale="0.001 0.001 0.001"/>
-        </geometry>
-        <material name="">
-          <color rgba="0.5 0.5 0.5 1"/>
-        </material>
-      </visual>
-      <inertial>
-        <mass value="0.1"/>
-        <origin xyz="0 0 0" rpy="0 0 0"/>
-        <inertia ixx="0.001" ixy="0.0" ixz="0.0"
-                 iyy="0.001" iyz="0.0"
-                 izz="0.001"/>
-      </inertial>
-    </link>
-    <link name="gs_cap_link">
-      <visual>
-        <geometry>
-          <mesh filename="package://gelsight_description/meshes/remain/gs_cap.stl" scale="0.001 0.001 0.001"/>
-        </geometry>
-        <material name="">
-          <color rgba="0 0 0 1"/>
-        </material>
-      </visual>
-      <inertial>
-        <mass value="0.1"/>
-        <origin xyz="0 0 0" rpy="0 0 0"/>
-        <inertia ixx="0.001" ixy="0.0" ixz="0.0"
-                 iyy="0.001" iyz="0.0"
-                 izz="0.001"/>
-      </inertial>
-    </link>
-    <!-- <link name="gs_gel_link">
-      <visual>
-        <geometry>
-          <mesh filename="package://gelsight_description/meshes/remain/gs_gel.stl" scale="0.001 0.001 0.001"/>
-        </geometry>
-        <material name="">
-            <color rgba="0.8 0.8 1.0 0.0"/>
-        </material>
-      </visual>
-      <inertial>
-        <mass value="0.1"/>
-        <origin xyz="0 0 0" rpy="0 0 0"/>
-        <inertia ixx="0.001" ixy="0.0" ixz="0.0"
-                 iyy="0.001" iyz="0.0"
-                 izz="0.001"/>
-      </inertial>
-    </link> -->
-      <link name="gs_gel_link">
-      <inertial>
-        <mass value="0.1"/>
-        <origin xyz="0 0 0" rpy="0 0 0"/>
-        <inertia ixx="0.001" ixy="0.0" ixz="0.0"
-                iyy="0.001" iyz="0.0"
-                izz="0.001"/>
-      </inertial>
-    </link>
-    <!-- <link name="gs_glass_link">
-      <visual>
-        <geometry>
-          <mesh filename="package://gelsight_description/meshes/remain/gs_glass.stl" scale="0.001 0.001 0.001"/>
-        </geometry>
-        <material name="">
-            <color rgba="1.0 1.0 1.0 0.3"/>
-        </material>
-      </visual>
-      <inertial>
-        <mass value="0.1"/>
-        <origin xyz="0 0 0" rpy="0 0 0"/>
-        <inertia ixx="0.001" ixy="0.0" ixz="0.0"
-                 iyy="0.001" iyz="0.0"
-                 izz="0.001"/>
-      </inertial>
-    </link> -->
-    <joint name="gs_holder_joint" type="fixed">
-      <parent link="${parent}"/>
-      <child link="gs_kinova_holder_link"/>
-      <origin xyz="-0.0380 -0.038 0" rpy="0 0 0"/>
-    </joint>
-    <joint name="gs_base_joint" type="fixed">
-      <parent link="${parent}"/>
-      <child link="gs_base_link"/>
-      <origin xyz="-0.014 -0.016 0" rpy="0 0 0"/>
-    </joint>
-    <joint name="gs_cap_joint" type="fixed">
-      <parent link="${parent}"/>
-      <child link="gs_cap_link"/>
-      <origin xyz="-0.0144 -0.016 0" rpy="0 0 0"/>
-    </joint>
-    <joint name="gs_gel_joint" type="fixed">
-      <parent link="${parent}"/>
-      <child link="gs_gel_link"/>
-      <origin xyz="-0.0115 -0.01386 0" rpy="0 0 0"/>
-    </joint>
-      <!-- +++++++++++++++++++++++camera link+++++++++++++++++++++++++++++ -->
-        <link name="gs_camera_link">
-      <visual>
-        <geometry>
-          <mesh filename="package://gelsight_description/meshes/remain/gs_glass.stl" scale="0.000001 0.0000001 0.0000001"/>
-        </geometry>
-      </visual>
-    </link>
-    <joint name="gs_camera_joint" type="fixed">
-      <parent link="gs_gel_link"/>
-      <child link="gs_camera_link"/>
-      <origin xyz="0.012 0.0143 0.035" rpy="0 ${-pi/2} ${pi}"/>
-      <!-- <origin xyz="0.0144 0.016 0.035" rpy="0 ${-pi/2} ${pi}"/> -->
-      <!-- <origin xyz="0.0 0.0 0.0" rpy="0 ${-pi/2} ${pi}"/> -->
-    </joint>
         <!-- <link name="fov_visual_link">
           <visual>
@@ -235,28 +209,4 @@
       <origin xyz="-0.0 -0.0 0" rpy="0 0 0"/>
     </joint> -->
-   <!-- + ++++++++++++++++++++++ Light simulation +++++++++++++++++++ -->
-   <!-- <gazebo reference="gs_gel_link">
-        <light type="point" name="led_left">
-            <pose>0.02 0 0 0 0 0</pose>
-            <diffuse>1.0 1.0 1.0 1</diffuse>
-            <attenuation>
-            <range>0.2</range>
-            <constant>0.5</constant>
-            <linear>0.01</linear>
-            <quadratic>0.001</quadratic>
-            </attenuation>
-        </light>
-        <light type="point" name="led_right">
-            <pose>-0.02 0 0 0 0 0</pose>
-            <diffuse>1.0 1.0 1.0 1</diffuse>
-            <attenuation>
-            <range>0.2</range>
-            <constant>0.5</constant>
-            <linear>0.01</linear>
-            <quadratic>0.001</quadratic>
-            </attenuation>
-        </light>
-        </gazebo> -->
-    <!-- ++++++++++++++++++++++++++++++++++++++++++++++++++++++++++ -->
     <xacro:gelsight_camera parent="gs_camera_link"/>
     <!-- <xacro:gelsight_spectre suffix="left" parent="gs_base_link" r="0" x="0.01" y="0" color="1 0 0"/>

File: src/gelsight_simulation_ros/gelsight_description/urdf/gs_mini_spectre.xacro (robot description, xacro)
@@ -13,5 +13,5 @@
       </visual>
       <inertial>
-        <mass value="0.01"/>
+        <mass value="0.2"/>
         <origin xyz="0 0 0" rpy="0 0 0"/>
         <inertia ixx="1e-5" ixy="0.0" ixz="0.0"
@@ -20,4 +20,5 @@
       </inertial>
     </link>
+    <!-- Colors of mirror leds -->
     <gazebo reference="gelsight_spectre_${suffix}">
       <visual>

Commit message: change gel position

File: src/gelsight_simulation_ros/gelsight_description/urdf/gelsight_sensor.xacro (robot description, xacro)
@@ -128,5 +128,5 @@
       <parent link="gs_gel_link"/>
       <child link="gs_camera_link"/>
-      <origin xyz="0.012 0.0143 0.035" rpy="0 ${-pi/2} ${pi}"/>
+      <origin xyz="0.0115 0.01386 0.035" rpy="0 ${-pi/2} ${pi}"/>
       <!-- <origin xyz="0.012 0.0143 0.035" rpy="0 0 0"/> -->
     </joint>
@@ -135,5 +135,5 @@
       <parent link="gs_gel_link"/>
       <child link="gs_camera_pcloud"/>
-      <origin xyz="0.012 0.0143 0.035" rpy="0 0 ${pi/2}"/>
+      <origin xyz="0.0115 0.01386 0.035" rpy="0 0 ${pi/2}"/>
     </joint>
      <!-- ++++++++++++++++++++++++++++++ Camera simulation +++++++++++++++++++++++++++++++++++-->
