Commit message: add gelsigth free body move

File: src/gelsight_simulation_ros/gelsight_description/urdf/gelsight_sensor_old.xacro (robot description, xacro)
@@ -1,5 +1,5 @@
 <?xml version="1.0"?>
 <robot xmlns:xacro="http://ros.org/wiki/xacro">
-  <xacro:include filename="$(find gelsight_description)/urdf/gs_mini_spectre.xacro"/>
+    zz<xacro:include filename="$(find gelsight_description)/urdf/gs_mini_spectre.xacro"/>
   <xacro:macro name="gelsight_sensor" params="parent">
     <link name="gs_kinova_holder_link">
@@ -54,5 +54,22 @@
       </inertial>
     </link>
-     <link name="gs_gel_link">
+    <!-- <link name="gs_gel_link">
+      <visual>
+        <geometry>
+          <mesh filename="package://gelsight_description/meshes/remain/gs_gel.stl" scale="0.001 0.001 0.001"/>
+        </geometry>
+        <material name="">
+            <color rgba="0.8 0.8 1.0 0.0"/>
+        </material>
+      </visual>
+      <inertial>
+        <mass value="0.1"/>
+        <origin xyz="0 0 0" rpy="0 0 0"/>
+        <inertia ixx="0.001" ixy="0.0" ixz="0.0"
+                 iyy="0.001" iyz="0.0"
+                 izz="0.001"/>
+      </inertial>
+    </link> -->
+      <link name="gs_gel_link">
       <inertial>
         <mass value="0.1"/>
@@ -63,5 +80,22 @@
       </inertial>
     </link>
-     <joint name="gs_holder_joint" type="fixed">
+    <!-- <link name="gs_glass_link">
+      <visual>
+        <geometry>
+          <mesh filename="package://gelsight_description/meshes/remain/gs_glass.stl" scale="0.001 0.001 0.001"/>
+        </geometry>
+        <material name="">
+            <color rgba="1.0 1.0 1.0 0.3"/>
+        </material>
+      </visual>
+      <inertial>
+        <mass value="0.1"/>
+        <origin xyz="0 0 0" rpy="0 0 0"/>
+        <inertia ixx="0.001" ixy="0.0" ixz="0.0"
+                 iyy="0.001" iyz="0.0"
+                 izz="0.001"/>
+      </inertial>
+    </link> -->
+    <joint name="gs_holder_joint" type="fixed">
       <parent link="${parent}"/>
       <child link="gs_kinova_holder_link"/>
@@ -84,5 +118,5 @@
     </joint>
       <!-- +++++++++++++++++++++++camera link+++++++++++++++++++++++++++++ -->
-     <link name="gs_camera_link">
+        <link name="gs_camera_link">
       <visual>
         <geometry>
@@ -95,4 +129,5 @@
       <child link="gs_camera_link"/>
       <origin xyz="0.012 0.0143 0.035" rpy="0 ${-pi/2} ${pi}"/>
+      <!-- <origin xyz="0.012 0.0143 0.035" rpy="0 0 0"/> -->
     </joint>
     <link name="gs_camera_pcloud"/>
@@ -136,5 +171,5 @@
           <depthImageInfoTopicName>/gelsight/depth/camera_info</depthImageInfoTopicName>
           <pointCloudTopicName>/gelsight/depth/points</pointCloudTopicName>
-          <frameName>gs_camera_link</frameName>
+          <frameName>gs_camera_pcloud</frameName>
           <pointCloudCutoff>0.0</pointCloudCutoff>
           <distortionK1>0</distortionK1>
@@ -152,9 +187,33 @@
     </gazebo>
   </xacro:macro>
+    <!-- +++++++++++++++++++++++++++++++++++++++++++++++++++++++++++++++++++++++++++++++++++ -->
+        <!-- <link name="fov_visual_link">
+          <visual>
+            <geometry>
+              <cylinder radius="0.005" length="0.3"/>
+            </geometry>
+            <material name="">
+              <color rgba="0 1 0 0.3"/>
+            </material>
+          </visual>
+        </link>
+        <joint name="fov_joint" type="fixed">
+          <parent link="gs_camera_link"/>
+          <child link="fov_visual_link"/>
+          <origin xyz="0 0 0.15" rpy="0 0 0"/>
+        </joint> -->
+      <!-- ++++++++++++++++++++++++++++++++++++++++++++++++++++++++++ -->
+     <!-- <joint name="gs_glass_link" type="fixed">
+      <parent link="${parent}"/>
+      <child link="gs_glass_link"/>
+      <origin xyz="-0.0 -0.0 0" rpy="0 0 0"/>
+    </joint> -->
     <xacro:gelsight_camera parent="gs_camera_link"/>
+    <!-- <xacro:gelsight_spectre suffix="left" parent="gs_base_link" r="0" x="0.01" y="0" color="1 0 0"/>
+    <xacro:gelsight_spectre suffix="right" parent="gs_base_link" r="0" x="-0.01" y="0" color="0 0 1"/> -->
     <xacro:gelsight_spectre suffix="bottom" parent="gs_base_link" color="1.0 1.0 1.0" r="0" x="-0.0235" y="-0.022" filename="package://gelsight_description/meshes/remain/spectre_bottom.stl"/>
     <xacro:gelsight_spectre suffix="right"  parent="gs_base_link" color="1.0 0.0 0.0" r="0" x="-0.0235" y="-0.022" filename="package://gelsight_description/meshes/remain/spectre_right.stl"/>
     <xacro:gelsight_spectre suffix="top"    parent="gs_base_link" color="0.0 1.0 0.0" r="0" x="-0.0235" y="-0.022" filename="package://gelsight_description/meshes/remain/spectre_top.stl"/>
     <xacro:gelsight_spectre suffix="left"   parent="gs_base_link" color="0.0 0.0 1.0" r="0" x="-0.0235" y="-0.022" filename="package://gelsight_description/meshes/remain/spectre_left.stl"/>
-  </xacro:macro>
+    </xacro:macro>
 </robot>
