Commit message: add files for simulation gelsight free

File: src/gelsight_simulation_ros/gelsight_description/urdf/gelsight_free.xacro (robot description, xacro)
@@ -6,10 +6,22 @@
   <link name="base_link">
     <inertial>
-      <mass value="0.001"/>
+      <mass value="0.1"/>
       <origin xyz="0 0 0" rpy="0 0 0"/>
-      <inertia ixx="1e-6" ixy="0.0" ixz="0.0"
-               iyy="1e-6" iyz="0.0"
-               izz="1e-6"/>
+      <inertia ixx="0.001" iyy="0.001" izz="0.001"
+              ixy="0.0" ixz="0.0" iyz="0.0"/>
     </inertial>
+        <visual>
+      <origin xyz="0 0 0" rpy="0 0 0"/>
+      <geometry>
+        <cylinder length="0.00001" radius="0.05"/>
+      </geometry>
+      <material name="Grey"/>
+    </visual>
+    <collision>
+      <origin xyz="0 0 0" rpy="0 0 0"/>
+      <geometry>
+        <cylinder length="0.00001" radius="0.05"/>
+      </geometry>
+</collision>
   </link>
   <!-- Instanciar el sensor físico -->

File: src/gelsight_simulation_ros/gelsight_description/urdf/gelsight_sensor.xacro (robot description, xacro)
@@ -136,5 +136,5 @@
           <depthImageInfoTopicName>/gelsight/depth/camera_info</depthImageInfoTopicName>
           <pointCloudTopicName>/gelsight/depth/points</pointCloudTopicName>
-          <frameName>gs_camera_link</frameName>
+          <frameName>gs_camera_pcloud</frameName>
           <pointCloudCutoff>0.0</pointCloudCutoff>
           <distortionK1>0</distortionK1>

Commit message: add new stl and fix errors whit velocity control on gs sesnor

File: src/gelsight_simulation_ros/gelsight_description/urdf/gelsight_free.xacro (robot description, xacro)
@@ -11,5 +11,5 @@
               ixy="0.0" ixz="0.0" iyz="0.0"/>
     </inertial>
-        <visual>
+        <!-- <visual>
       <origin xyz="0 0 0" rpy="0 0 0"/>
       <geometry>
@@ -23,5 +23,5 @@
         <cylinder length="0.00001" radius="0.05"/>
       </geometry>
-</collision>
+</collision> -->
   </link>
   <!-- Instanciar el sensor físico -->
@@ -32,5 +32,4 @@
   </gazebo>
 <gazebo>
-  <!-- <plugin name="gelsight_force_move" filename="libgazebo_ros_force_based_move.so"> -->
   <plugin name="apply_force" filename="libgazebo_ros_force.so">
     <bodyName>base_link</bodyName>

File: src/gelsight_simulation_ros/gelsight_description/urdf/gelsight_sensor.xacro (robot description, xacro)
@@ -66,20 +66,20 @@
       <parent link="${parent}"/>
       <child link="gs_kinova_holder_link"/>
-      <origin xyz="-0.0380 -0.038 0" rpy="0 0 0"/>
+      <origin xyz="0.0 0.0 0.0127151" rpy="0 0 0"/>
     </joint>
     <joint name="gs_base_joint" type="fixed">
-      <parent link="${parent}"/>
+      <parent link="gs_kinova_holder_link"/>
       <child link="gs_base_link"/>
-      <origin xyz="-0.014 -0.016 0" rpy="0 0 0"/>
+      <origin xyz="0.0 0.0 0.0205405" rpy="0 0 0"/>
     </joint>
     <joint name="gs_cap_joint" type="fixed">
-      <parent link="${parent}"/>
+      <parent link="gs_base_link"/>
       <child link="gs_cap_link"/>
-      <origin xyz="-0.0144 -0.016 0" rpy="0 0 0"/>
+      <origin xyz="0.0 0.0 0.0129196" rpy="0 0 0"/>
     </joint>
     <joint name="gs_gel_joint" type="fixed">
-      <parent link="${parent}"/>
+      <parent link="gs_base_link"/>
       <child link="gs_gel_link"/>
-      <origin xyz="-0.0115 -0.01386 0" rpy="0 0 0"/>
+      <origin xyz="0.0 0.0 0.0184587" rpy="0 0 0"/>
     </joint>
       <!-- +++++++++++++++++++++++camera link+++++++++++++++++++++++++++++ -->
@@ -92,13 +92,13 @@
     </link>
     <joint name="gs_camera_joint" type="fixed">
-      <parent link="gs_gel_link"/>
+      <parent link="gs_base_link"/>
       <child link="gs_camera_link"/>
-      <origin xyz="0.012 0.0143 0.035" rpy="0 ${-pi/2} ${pi}"/>
+      <origin xyz="0.0 0.0 0.00154" rpy="0 ${-pi/2} ${pi}"/>
     </joint>
     <link name="gs_camera_pcloud"/>
     <joint name="gs_camera_pcloud_joint" type="fixed">
-      <parent link="gs_gel_link"/>
+      <parent link="gs_base_link"/>
       <child link="gs_camera_pcloud"/>
-      <origin xyz="0.0115 0.01386 0.035" rpy="0 0 ${pi/2}"/>
+      <origin xyz="0.0 0.0 0.00154" rpy="0 0 ${pi/2}"/>
     </joint>
      <!-- ++++++++++++++++++++++++++++++ Camera simulation +++++++++++++++++++++++++++++++++++-->
@@ -153,8 +153,8 @@
   </xacro:macro>
     <xacro:gelsight_camera parent="gs_camera_link"/>
-    <xacro:gelsight_spectre suffix="bottom" parent="gs_base_link" color="1.0 1.0 1.0" r="0" x="-0.0235" y="-0.022" filename="package://gelsight_description/meshes/remain/spectre_bottom.stl"/>
-    <xacro:gelsight_spectre suffix="right"  parent="gs_base_link" color="1.0 0.0 0.0" r="0" x="-0.0235" y="-0.022" filename="package://gelsight_description/meshes/remain/spectre_right.stl"/>
-    <xacro:gelsight_spectre suffix="top"    parent="gs_base_link" color="0.0 1.0 0.0" r="0" x="-0.0235" y="-0.022" filename="package://gelsight_description/meshes/remain/spectre_top.stl"/>
-    <xacro:gelsight_spectre suffix="left"   parent="gs_base_link" color="0.0 0.0 1.0" r="0" x="-0.0235" y="-0.022" filename="package://gelsight_description/meshes/remain/spectre_left.stl"/>
+    <xacro:gelsight_spectre suffix="bottom" parent="gs_base_link" color="1.0 1.0 1.0" r="0" x=" 0.0" y="-0.012" filename="package://gelsight_description/meshes/remain/spectre_bottom.stl"/>
+    <xacro:gelsight_spectre suffix="right"  parent="gs_base_link" color="1.0 0.0 0.0" r="0" x=" 0.009" y=" 0.0" filename="package://gelsight_description/meshes/remain/spectre_right.stl"/>
+    <xacro:gelsight_spectre suffix="top"    parent="gs_base_link" color="0.0 1.0 0.0" r="0" x=" 0.0" y=" 0.012" filename="package://gelsight_description/meshes/remain/spectre_top.stl"/>
+    <xacro:gelsight_spectre suffix="left"   parent="gs_base_link" color="0.0 0.0 1.0" r="0" x="-0.009" y=" 0.0" filename="package://gelsight_description/meshes/remain/spectre_left.stl"/>
   </xacro:macro>
 </robot>

File: src/gelsight_simulation_ros/gelsight_description/urdf/gs_mini_spectre.xacro (robot description, xacro)
@@ -4,5 +4,5 @@
     <link name="gelsight_spectre_${suffix}">
       <visual>
-        <origin rpy="0 0 ${r}" xyz="${x} ${y} 0.0"/>
+        <origin rpy="0 0 ${r}" xyz="${x} ${y} 0.0129294"/>
         <geometry>
           <mesh filename="${filename}" scale="0.001 0.001 0.001"/>
@@ -13,5 +13,5 @@
       </visual>
       <inertial>
-        <mass value="0.2"/>
+        <mass value="0.01"/>
         <origin xyz="0 0 0" rpy="0 0 0"/>
         <inertia ixx="1e-5" ixy="0.0" ixz="0.0"
