Commit message: change twist velocity frame to the gs_camera_pcloud frame, and add the description on readme

File: src/gelsight_simulation_ros/gelsight_description/urdf/gelsight_sensor_holder.xacro (robot description, xacro)
@@ -63,13 +63,19 @@
       </inertial>
     </link>
-     <joint name="gs_holder_joint" type="fixed">
+    <link name="gs_camera_pcloud"/>
+    <joint name="gs_camera_pcloud_joint" type="fixed">
       <parent link="${parent}"/>
-      <child link="gs_kinova_holder_link"/>
-      <origin xyz="0.0 0.0 0.0127151" rpy="0 0 0"/>
+      <child link="gs_camera_pcloud"/>
+      <origin xyz="0.0 0.0 0.035" rpy="0 0 1.571"/>
+    </joint>
+    <joint name="gs_camera_base_joint" type="fixed">
+      <parent link="gs_camera_pcloud"/>
+      <child link="gs_base_link"/>
+      <origin xyz="0.0 0.0 -0.00154" rpy="0 0 -${pi/2}"/>
     </joint>
     <joint name="gs_base_joint" type="fixed">
-      <parent link="gs_kinova_holder_link"/>
-      <child link="gs_base_link"/>
-      <origin xyz="0.0 0.0 0.0205405" rpy="0 0 0"/>
+      <parent link="gs_base_link"/>
+      <child link="gs_kinova_holder_link"/>
+      <origin xyz="0.0 0.0 -0.0205405" rpy="0 0 0"/>
     </joint>
     <joint name="gs_cap_joint" type="fixed">
@@ -96,10 +102,10 @@
       <origin xyz="0.0 0.0 0.00154" rpy="0 ${-pi/2} ${pi}"/>
     </joint>
-    <link name="gs_camera_pcloud"/>
+    <!-- <link name="gs_camera_pcloud"/>
     <joint name="gs_camera_pcloud_joint" type="fixed">
       <parent link="gs_base_link"/>
       <child link="gs_camera_pcloud"/>
       <origin xyz="0.0 0.0 0.00154" rpy="0 0 ${pi/2}"/>
-    </joint>
+    </joint> -->
      <!-- ++++++++++++++++++++++++++++++ Camera simulation +++++++++++++++++++++++++++++++++++-->
      <xacro:macro name="gelsight_camera" params="parent">

File: src/gelsight_simulation_ros/gelsight_description/urdf/gelsight_twist_link.xacro (robot description, xacro)
@@ -2,5 +2,5 @@
 <robot xmlns:xacro="http://ros.org/wiki/xacro" name="gelsight_sensor">
   <!-- Incluir la macro principal -->
-  <xacro:include filename="$(find gelsight_description)/urdf/gelsight_sensor.xacro" />
+  <xacro:include filename="$(find gelsight_description)/urdf/gelsight_sensor_free_body.xacro" />
   <!-- Definir base_link -->
   <link name="base_link">

File: src/ros_kortex/kortex_description/robots/gs_kinova_robot.xacro (robot description, xacro)
@@ -51,5 +51,5 @@
           </material>
     <!-- +++++++++++++++++++++++++++++++++++++++++++++++++++++GS mini +++++++++++++++++++++++++++++++++++++++++++++++++++++++++ -->
-<xacro:include filename="$(find gelsight_description)/urdf/gelsight_sensor.xacro"/>
+<xacro:include filename="$(find gelsight_description)/urdf/gelsight_sensor_holder.xacro"/>
 <xacro:gelsight_sensor parent="tool_frame"/>
 <!-- ++++++++++++++++++++++++++++++++++++++++++++++++++++++++++++++++++++++++++++++++++++++++++++++++++++++++++++++++++++++++++++	 -->
