Commit message: rotate the sensor to aline with kinova end efector frame

File: src/ros_kortex/kortex_description/robots/gs_kinova_robot.xacro (robot description, xacro)
@@ -38,5 +38,5 @@
             <link name="${prefix}tool_frame"/>
             <joint name="${prefix}tool_frame_joint" type="fixed">
-                <origin xyz="0 0 0" rpy="0 0 0" />
+                <origin xyz="0 0 0" rpy="0 0 -1.57" />
                 <parent link="${prefix}${last_arm_link}" />
                 <child link="${prefix}tool_frame" />
